File: ISOish88.kicad_pcb (KiCad board)
At the start: 2 copper layers, 344.6 x 125.9 mm, 288 parts, among them J1 Conn_01x04_Pin, J3 USB_C_Receptacle_USB2.0_14P, K1 Esc, K10 F9, K11 F10, K12 F11, K13 F12, K14 Print, K15 Scroll, K16 Pause, K17 ` ~, K18 1, K19 2, K2 F1, K20 3, K21 4, K22 5, K23 6, K24 7, K25 8, K26 9, K27 0, K28 - _, K29 = +, K3 F2, K30 Backspace, K31 Ins, K32 Home, K33 PgUp, K34 Tab, K35 Q, K36 W, K37 E, K38 R, K39 T, K4 F3, K40 Y, K41 U, K42 I, K43 O, K44 P, K45 [ {, K46 ] }, K47 Enter, K48 Del, K49 End, K5 F4, K50 PgDn, K51 Caps, K52 A, K53 S, K54 D, K55 F, K56 G, K57 H, K58 J, K59 K, K6 F5, K60 L, K61 ; :, K62 ' ", K63 \ |, K64 LShift, K65 Z, K66 X, K67 C, K68 V, K69 B, K7 F6, K70 N, K71 M, K72 , <, K73 . >, K74 / ?, K75 SplitRShift, K76 Fn, K77 Up, K78 LCtrl, K79 LSys, K8 F7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

Commit message: more RGB footprint fixes
Parts:
- moved FID3 1.00 mm to (347.7, 106.3)
Connections:
- BD1 pad 1: +5V -> Net-(BD1-VDD)
- BD1 pad 2: Net-(BD1-DOUT) -> GND
- BD1 pad 3: GND -> Net-(BD1-VSS)
- BD1 pad 4: Net-(BD1-DIN) -> +5V
- BD10 pad 1: +5V -> Net-(BD10-VDD)
- BD10 pad 2: Net-(BD10-DOUT) -> GND
- BD10 pad 3: GND -> Net-(BD10-VSS)
- BD10 pad 4: Net-(BD10-DIN) -> +5V
- BD11 pad 1: +5V -> Net-(BD11-VDD)
- BD11 pad 2: Net-(BD10-DIN) -> GND
- BD11 pad 3: GND -> Net-(BD10-VDD)
- BD11 pad 4: Net-(BD11-DIN) -> +5V
- BD12 pad 1: +5V -> Net-(BD12-VDD)
- BD12 pad 2: Net-(BD11-DIN) -> GND
- BD12 pad 3: GND -> Net-(BD11-VDD)
- BD12 pad 4: Net-(BD12-DIN) -> +5V
- BD13 pad 1: +5V -> Net-(BD13-VDD)
- BD13 pad 2: Net-(BD12-DIN) -> GND
- BD13 pad 3: GND -> Net-(BD12-VDD)
- BD13 pad 4: Net-(BD13-DIN) -> +5V
- BD14 pad 1: +5V -> Net-(BD14-VDD)
- BD14 pad 2: Net-(BD13-DIN) -> GND
- BD14 pad 3: GND -> Net-(BD13-VDD)
- BD14 pad 4: Net-(BD14-DIN) -> +5V
- BD15 pad 1: +5V -> Net-(BD15-DOUT)
- BD15 pad 2: Net-(BD14-DIN) -> GND
- BD15 pad 3: GND -> Net-(BD14-VDD)
- BD15 pad 4: Net-(BD15-DIN) -> +5V
- BD16 pad 1: +5V -> unconnected-(BD16-DOUT-Pad1)
- BD16 pad 2: Net-(BD15-DIN) -> GND
- BD16 pad 3: GND -> Net-(BD15-DOUT)
- BD16 pad 4: unconnected-(BD16-DIN-Pad4) -> +5V
- BD2 pad 1: +5V -> Net-(BD2-VDD)
- BD2 pad 2: Net-(BD1-DIN) -> GND
- BD2 pad 3: GND -> Net-(BD1-VDD)
- BD2 pad 4: Net-(BD2-DIN) -> +5V
- BD3 pad 1: +5V -> Net-(BD3-VDD)
- BD3 pad 2: Net-(BD2-DIN) -> GND
- BD3 pad 3: GND -> Net-(BD2-VDD)
- BD3 pad 4: Net-(BD3-DIN) -> +5V
- BD4 pad 1: +5V -> Net-(BD4-VDD)
- BD4 pad 2: Net-(BD3-DIN) -> GND
- BD4 pad 3: GND -> Net-(BD3-VDD)
- BD4 pad 4: Net-(BD4-DIN) -> +5V
- BD5 pad 1: +5V -> Net-(BD5-VDD)
- BD5 pad 2: Net-(BD4-DIN) -> GND
- BD5 pad 3: GND -> Net-(BD4-VDD)
- BD5 pad 4: Net-(BD5-DIN) -> +5V
- BD6 pad 1: +5V -> Net-(BD6-VDD)
- BD6 pad 2: Net-(BD5-DIN) -> GND
- BD6 pad 3: GND -> Net-(BD5-VDD)
- BD6 pad 4: Net-(BD6-DIN) -> +5V
- BD7 pad 1: +5V -> Net-(BD7-VDD)
- BD7 pad 2: Net-(BD6-DIN) -> GND
- BD7 pad 3: GND -> Net-(BD6-VDD)
- BD7 pad 4: Net-(BD7-DIN) -> +5V
- BD8 pad 1: +5V -> Net-(BD8-VDD)
- BD8 pad 2: Net-(BD7-DIN) -> GND
- BD8 pad 3: GND -> Net-(BD7-VDD)
- BD8 pad 4: Net-(BD8-DIN) -> +5V
- BD9 pad 1: +5V -> Net-(BD10-VSS)
- BD9 pad 2: Net-(BD8-DIN) -> GND
- BD9 pad 3: GND -> Net-(BD8-VDD)
- BD9 pad 4: Net-(BD10-DOUT) -> +5V
- JP1 pad 3: Net-(BD1-DOUT) -> Net-(BD1-VSS)
- LD78 pad 2: Net-(BD1-DOUT) -> Net-(BD1-VSS)
Routing:
- net Net-(BD1-DOUT): track 111.2 -> 0.00 mm, vias 3 -> 0
- net Net-(BD1-VSS): track 0.00 -> 109.1 mm, vias 0 -> 3
- net Net-(BD8-VDD): track 0.00 -> 89.9 mm
- net Net-(BD8-DIN): track 88.8 -> 0.00 mm
- net Net-(BD15-DOUT): track 0.00 -> 66.0 mm, vias 0 -> 2
- net Net-(BD1-VDD): track 0.00 -> 61.5 mm, vias 0 -> 2
- net Net-(BD10-VDD): track 0.00 -> 60.1 mm, vias 0 -> 4
- net Net-(BD5-VDD): track 0.00 -> 57.4 mm, vias 0 -> 2
- net Net-(BD10-VSS): track 0.00 -> 57.0 mm, vias 0 -> 4
- net Net-(BD4-VDD): track 0.00 -> 56.6 mm, vias 0 -> 2
- net Net-(BD3-VDD): track 0.00 -> 56.6 mm, vias 0 -> 2
- net Net-(BD7-VDD): track 0.00 -> 56.4 mm, vias 0 -> 4
- net Net-(BD2-VDD): track 0.00 -> 56.0 mm, vias 0 -> 2
- net Net-(BD11-VDD): track 0.00 -> 56.0 mm, vias 0 -> 2
- net Net-(BD6-VDD): track 0.00 -> 55.6 mm, vias 0 -> 2
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