File: ISOish88.kicad_pcb (KiCad board)
At the start: 2 copper layers, 344.6 x 125.9 mm, 288 parts, among them J1 Conn_01x04_Pin, J3 USB_C_Receptacle_USB2.0_14P, K1 Esc, K10 F9, K11 F10, K12 F11, K13 F12, K14 Print, K15 Scroll, K16 Pause, K17 ` ~, K18 1, K19 2, K2 F1, K20 3, K21 4, K22 5, K23 6, K24 7, K25 8, K26 9, K27 0, K28 - _, K29 = +, K3 F2, K30 Backspace, K31 Ins, K32 Home, K33 PgUp, K34 Tab, K35 Q, K36 W, K37 E, K38 R, K39 T, K4 F3, K40 Y, K41 U, K42 I, K43 O, K44 P, K45 [ {, K46 ] }, K47 Enter, K48 Del, K49 End, K5 F4, K50 PgDn, K51 Caps, K52 A, K53 S, K54 D, K55 F, K56 G, K57 H, K58 J, K59 K, K6 F5, K60 L, K61 ; :, K62 ' ", K63 \ |, K64 LShift, K65 Z, K66 X, K67 C, K68 V, K69 B, K7 F6, K70 N, K71 M, K72 , <, K73 . >, K74 / ?, K75 SplitRShift, K76 Fn, K77 Up, K78 LCtrl, K79 LSys, K8 F7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

Commit message: tweaks
Parts:
- added C10: 1u, schizobovine:C_0603_1608Metric, B.Cu at (81.0, 109.5)
- added C17: 1u, schizobovine:C_0603_1608Metric, B.Cu at (71.8, 132.2)
- added C18: 1u, schizobovine:C_0603_1608Metric, B.Cu at (81.7, 144.7)
- added C7: 1u, schizobovine:C_0603_1608Metric, B.Cu at (66.6, 71.5)
- added C8: 1u, schizobovine:C_0603_1608Metric, B.Cu at (76.2, 90.1)
- C12: value 1u -> 4u7; footprint schizobovine:C_0603_1608Metric -> schizobovine:C_0805_2012Metric
- H1, H2, H3, H4: footprint schizobovine:MountingHole_2.2mm_M2_Pad_TopOnly -> schizobovine:MountingHole_3.0mm_M2_5mm_dia_solderable
- U5: footprint MCU_RaspberryPi_and_Boards:RP2040-QFN-56 -> schizobovine:RP2040-QFN-56
Routing:
- net +5V: track 2375.1 -> 2381.8 mm, vias 118 -> 123
- net row1: track 449.1 -> 455.4 mm
- net row0: track 397.5 -> 400.8 mm, vias 12 -> 10
- net rgb_3v3: track 354.1 -> 356.2 mm
- net row2: track 410.7 -> 411.8 mm
Other:
- board text added: "MAXX"
- board text added: "RGB?"
- board text added: "Underglow ONLY"
- board text added: "v1.1"
- board text removed: "v1.0"
